File: Hardware/Contact Mic Board/Contact Mic Board.kicad_sch (KiCad schematic)
At the start: 47 parts, among them J1 Conn_01x09_Pin, U1 ES8388, U2 MCP6002-xMC

Commit message: received feedback from Andy + others and revised board
Parts:
- added C20: 10uF, Capacitor_SMD:C_0402_1005Metric, symbol Device:C_Polarized_Small_US
Connections:
- net +3.3V: now also C20.1
- net GND: now also C20.2
Other:
- moved on the sheet: TP2
