File: Hardware/Main Board/Main Board.kicad_sch (KiCad schematic)
At the start: 85 parts, among them J1 Micro_SD_Card_Det1, J3 Conn_01x09_Socket, J4 MIC 1 Connector, J5 MIC 2 Connector, J6 USB_C_Receptacle_USB2.0_16P, J7 OLED, Q1 AO3401A, SW1 SW_SPST, U1 ESP32-S3-WROOM-2, U2 TPS63060, U3 TP4056-42-ESOP8, U4 TLV75528PDBV, U6 AP2112K-1.2

Commit message: submitted for manufacturing
Parts:
- D1: footprint LED_SMD:LED_0603_1608Metric -> Connector_PinHeader_2.54mm:PinHeader_1x02_P2.54mm_Vertical
- R11: value 10k -> 4.7k
- R13, R14: value 4.7k -> 10k
- renumbered TP2 to 3V3, TP5 to BATT1, TP1 to GND1
Connections:
- net +3.3V: now also 600Ω@100MHz1.1; no longer C20.1, U4.1 (IN)
- net 2.8V: now also C21.1, U4.5 (OUT); no longer 600Ω@100MHz1.2
- new net: 600Ω@100MHz1.2, C20.1, U4.1 (IN)
Other:
- moved on the sheet: 600Ω@100MHz1, A2V8, C20
Changed lines of the file:
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@@
 	)
 	(junction
-		(at 308.61 215.9)
-		(diameter 0)
-		(color 0 0 0 0)
-	)
-	(junction
 		(at 69.85 184.15)
 		(diameter 0)
@@
 	)
 	(junction
-		(at 30.48 52.07)
+		(at 308.61 215.9)
 		(diameter 0)
 		(color 0 0 0 0)
 	)
 	(junction
-		(at 148.59 73.66)
+		(at 30.48 52.07)
 		(diameter 0)
 		(color 0 0 0 0)
 	)
 	(junction
-		(at 325.12 215.9)
+		(at 148.59 73.66)
 		(diameter 0)
 		(color 0 0 0 0)
@@
 	)
 	(junction
+		(at 317.5 215.9)
+		(diameter 0)
+		(color 0 0 0 0)
+	)
+	(junction
 		(at 39.37 173.99)
 		(diameter 0)
@@
 	(wire
 		(pts
-			(xy 323.85 215.9) (xy 325.12 215.9)
+			(xy 279.4 215.9) (xy 287.02 215.9)
 		)
 		(stroke
@@
 	(wire
 		(pts
-			(xy 284.48 215.9) (xy 287.02 215.9)
+			(xy 270.51 215.9) (xy 271.78 215.9)
 		)
 		(stroke
@@
 	(wire
 		(pts
-			(xy 308.61 215.9) (xy 316.23 215.9)
+			(xy 58.42 184.15) (xy 69.85 184.15)
 		)
 		(stroke
@@
 	(wire
 		(pts
-			(xy 58.42 184.15) (xy 69.85 184.15)
+			(xy 39.37 179.07) (xy 44.45 179.07)
 		)
 		(stroke
@@
 	(wire
 		(pts
-			(xy 39.37 179.07) (xy 44.45 179.07)
+			(xy 69.85 184.15) (xy 69.85 189.23)
 		)
 		(stroke
@@
 	(wire
 		(pts
-			(xy 69.85 184.15) (xy 69.85 189.23)
+			(xy 304.8 185.42) (xy 304.8 187.96)
 		)
 		(stroke
@@
 	(wire
 		(pts
-			(xy 304.8 185.42) (xy 304.8 187.96)
+			(xy 125.73 73.66) (xy 127 73.66)
 		)
 		(stroke
@@
 	(wire
 		(pts
-			(xy 125.73 73.66) (xy 127 73.66)
+			(xy 287.02 214.63) (xy 287.02 215.9)
 		)
 		(stroke
@@
 	(wire
 		(pts
-			(xy 287.02 213.36) (xy 287.02 215.9)
+			(xy 173.99 35.56) (xy 173.99 43.18)
 		)
 		(stroke
@@
 	(wire
 		(pts
-			(xy 173.99 35.56) (xy 173.99 43.18)
+			(xy 308.61 215.9) (xy 317.5 215.9)
 		)
 		(stroke
@@
 	(wire
 		(pts
-			(xy 325.12 215.9) (xy 327.66 215.9)
+			(xy 317.5 215.9) (xy 320.04 215.9)
 		)
 		(stroke
@@
 	(global_label "2.8V"
 		(shape input)
-		(at 327.66 215.9 0)
+		(at 320.04 215.9 0)
 		(fields_autoplaced yes)
 		(effects
@@
 		)
 		(property "Intersheetrefs" "${INTERSHEET_REFS}"
-			(at 334.7576 215.9 0)
+			(at 327.1376 215.9 0)
 			(effects
 				(font
@@
 			)
 		)
-		(property "Value" "4.7k"
+		(property "Value" "10k"
 			(at 155.194 46.736 90)
 			(effects
@@
 		(dnp no)
 		(fields_autoplaced yes)
-		(property "Reference" "TP1"
-			(at 48.26 20.8279 0)
+		(property "Reference" "GND1"
+			(at 48.26 22.0979 0)
 			(effects
 				(font
@@
 			(project "Main Board"
 				(path "/06300a21-1646-41b0-b473-1c39557d6dab"
-					(reference "TP1")
+					(reference "GND1")
 					(unit 1)
 				)
@@
 	(symbol
 		(lib_id "power:GND")
-		(at 287.02 208.28 180)
+		(at 287.02 209.55 180)
 		(unit 1)
 		(exclude_from_sim no)
@@
 		(fields_autoplaced yes)
 		(property "Reference" "#PWR083"
-			(at 287.02 201.93 0)
+			(at 287.02 203.2 0)
 			(effects
 				(font
@@
 		)
 		(property "Value" "GND"
-			(at 287.02 203.2 0)
+			(at 287.02 204.47 0)
 			(effects
 				(font
@@
 		)
 		(property "Footprint" ""
-			(at 287.02 208.28 0)
+			(at 287.02 209.55 0)
 			(effects
 				(font
@@
 		)
 		(property "Datasheet" ""
-			(at 287.02 208.28 0)
+			(at 287.02 209.55 0)
 			(effects
 				(font
@@
 		)
 		(property "Description" "Power symbol creates a global label with name \"GND\" , ground"
-			(at 287.02 208.28 0)
+			(at 287.02 209.55 0)
 			(effects
 				(font
@@
 		(dnp no)
 		(fields_autoplaced yes)
-		(property "Reference" "TP5"
+		(property "Reference" "BATT1"
 			(at 207.01 46.4819 0)
 			(effects
@@
 			(project "Main Board"
 				(path "/06300a21-1646-41b0-b473-1c39557d6dab"
-					(reference "TP5")
+					(reference "BATT1")
 					(unit 1)
 				)
@@
 			)
 		)
-		(property "Footprint" "LED_SMD:LED_0603_1608Metric"
+		(property "Footprint" "Connector_PinHeader_2.54mm:PinHeader_1x02_P2.54mm_Vertical"
 			(at 88.9 40.64 0)
 			(effects
@@
 			)
 		)
-		(property "Value" "4.7k"
+		(property "Value" "10k"
 			(at 155.194 56.896 90)
 			(effects
@@
 	(symbol
 		(lib_id "Device:C_Small")
-		(at 287.02 210.82 180)
+		(at 287.02 212.09 180)
 		(unit 1)
 		(exclude_from_sim no)
@@
 		(dnp no)
 		(property "Reference" "C20"
-			(at 291.846 212.852 0)
+			(at 291.846 214.122 0)
 			(effects
 				(font
@@
 		)
 		(property "Value" "1uF"
-			(at 293.37 210.82 0)
+			(at 293.37 212.09 0)
 			(effects
 				(font
@@
 		)
 		(property "Footprint" "Capacitor_SMD:C_0603_1608Metric"
-			(at 287.02 210.82 0)
+			(at 287.02 212.09 0)
 			(effects
 				(font
@@
 		)
 		(property "Datasheet" "~"
-			(at 287.02 210.82 0)
+			(at 287.02 212.09 0)
 			(effects
 				(font
@@
 		)
 		(property "Description" "Unpolarized capacitor, small symbol"
-			(at 287.02 210.82 0)
+			(at 287.02 212.09 0)
 			(effects
 				(font
@@
 			)
 		)
-		(property "Value" "10k"
+		(property "Value" "4.7k"
 			(at 86.614 48.514 90)
 			(effects
@@
 	(symbol
 		(lib_id "Connector:TestPoint")
-		(at 325.12 215.9 180)
+		(at 317.5 215.9 180)
 		(unit 1)
 		(exclude_from_sim no)
@@
 		(dnp no)
 		(property "Reference" "A2V8"
-			(at 330.454 221.742 0)
+			(at 322.834 221.742 0)
 			(effects
 				(font
@@
 		)
 		(property "Value" "TestPoint"
-			(at 322.58 217.9321 0)
+			(at 314.96 217.9321 0)
 			(effects
 				(font
@@
 		)
 		(property "Footprint" "TestPoint:TestPoint_Pad_1.0x1.0mm"
-			(at 320.04 215.9 0)
+			(at 312.42 215.9 0)
 			(effects
 				(font
@@
 		)
 		(property "Datasheet" "~"
-			(at 320.04 215.9 0)
+			(at 312.42 215.9 0)
 			(effects
 				(font
@@
 		)
 		(property "Description" "test point"
-			(at 325.12 215.9 0)
+			(at 317.5 215.9 0)
 			(effects
 				(font
@@
 		(dnp no)
 		(fields_autoplaced yes)
-		(property "Reference" "TP2"
-			(at 62.23 32.2579 0)
+		(property "Reference" "3V3"
+			(at 62.23 33.5279 0)
 			(effects
 				(font
@@
 			(project ""
 				(path "/06300a21-1646-41b0-b473-1c39557d6dab"
-					(reference "TP2")
+					(reference "3V3")
 					(unit 1)
 				)
@@
 	(symbol
 		(lib_id "Device:FerriteBead")
-		(at 320.04 215.9 90)
+		(at 275.59 215.9 90)
 		(unit 1)
 		(exclude_from_sim no)
@@
 		(fields_autoplaced yes)
 		(property "Reference" "600Ω@100MHz1"
-			(at 319.9892 208.28 90)
+			(at 275.5392 208.28 90)
 			(effects
 				(font
@@
 		)
 		(property "Value" "FerriteBead"
-			(at 319.9892 210.82 90)
+			(at 275.5392 210.82 90)
 			(effects
 				(font
@@
 		)
 		(property "Footprint" "Resistor_SMD:R_0603_1608Metric"
-			(at 320.04 217.678 90)
+			(at 275.59 217.678 90)
 			(effects
 				(font
@@
 		)
 		(property "Datasheet" "~"
-			(at 320.04 215.9 0)
+			(at 275.59 215.9 0)
 			(effects
 				(font
@@
 		)
 		(property "Description" "Ferrite bead"
-			(at 320.04 215.9 0)
+			(at 275.59 215.9 0)
 			(effects
 				(font
@@
 	(symbol
 		(lib_id "power:+3.3V")
-		(at 284.48 215.9 90)
+		(at 270.51 215.9 90)
 		(unit 1)
 		(exclude_from_sim no)
@@
 		(dnp no)
 		(property "Reference" "#PWR069"
-			(at 288.29 215.9 0)
+			(at 274.32 215.9 0)
 			(effects
 				(font
@@
 		)
 		(property "Value" "+3.3V"
-			(at 278.13 215.9 90)
+			(at 264.16 215.9 90)
 			(effects
 				(font
@@
 		)
 		(property "Footprint" ""
-			(at 284.48 215.9 0)
+			(at 270.51 215.9 0)
 			(effects
 				(font
@@
 		)
 		(property "Datasheet" ""
-			(at 284.48 215.9 0)
+			(at 270.51 215.9 0)
 			(effects
 				(font
@@
 		)
 		(property "Description" "Power symbol creates a global label with name \"+3.3V\""
-			(at 284.48 215.9 0)
+			(at 270.51 215.9 0)
 			(effects
 				(font
